File: CM4 Shield/CM4_shield.sch (EAGLE design)
At the start: 39 parts, among them J1 TERMINALBLOCK/TOYO/2PIN/5MMPI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, J3 RASPBERRYPI-40-PIN-GPIO_PTH_N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, X4 DOOR LOCK, X6 TOWER LIGHT

Commit message: update to board design
Parts:
- removed FWLOGO_1: FWLOGO, FracktalWorks:FWLOGO
- removed J1: TERMINALBLOCK/TOYO/2PIN/5MMPITCH, FracktalWorks:TERMINALBLOCK/TOYO/2PIN/5MMPITCH
- added J4: 2828XX-2282837-2, Connector:2828XX-2282837-2
- added TP3: TEST-POINT3X5, SparkFun-Connectors:TEST-POINT3X5
- added X1: JST-XH-02-PIN-LONG-PAD, Rembrandt Electronics - JST XH Connectors v1-0:JST-XH-02-PIN-LONG-PAD
Connections:
- new net BUZZER: J3.GP12, TP3.1, X1-1.S
- net +24V: now also J4.1; no longer J1.1
- net GND: now also J4.2, X1-2.S; no longer J1.2
Other:
- moved on the sheet: J3, X4-1, X4-2, X4-3, X6-1, X6-2, X6-3, X6-4
